Commit message: feat(sim): add crossing obstacle experiment scene

File: src/my_tb3_description/urdf_w_sensor/turtlebot3_burger.urdf.xacro (robot description, xacro)
@@ -55,5 +55,5 @@
   <!-- D435 camera -->
   <xacro:sensor_d435 name="d435" parent="base_link" use_mesh="true" use_nominal_extrinsics="true">
-    <origin xyz="0 0 0.18" rpy="0 0 0" />
+    <origin xyz="0 0 0.18" rpy="0 -0.2 0" />
   </xacro:sensor_d435>
   <joint name="wheel_left_joint" type="continuous">
