Commit message: real_world_exp: DOA perception + T-MPC planner for real robot deployment
Core components:
- DOA: RGB-D perception pipeline (SAM + CLIP + rematch + pointcloud)
- mpc_planner: C++ T-MPC framework (Acados solver, GMM uncertainty)
- mpc_planner_jackalsimulator: ROS1 planner node (no Gazebo runtime dep)
- guidance_planner: topology-aware global planning (Visibility-PRM)
- roadmap + roadmap_msgs: XML/YAML map to spline reference paths
- ros_tools: shared C++ utilities (visualization, logging, math)
- DecompUtil: ellipsoid decomposition for static obstacle constraints
- asr_rapidxml: RapidXML ROS wrapper (roadmap dependency)
- catkin_simple: build helper

Bridge and config:
- doa_to_tmpc.py: DOA TrackerDetailArray -> mpc_planner_msgs/ObstacleArray
- doa_to_obstacles.py: DOA -> Python MPC bridge (baseline reference)
- mpc.yaml, mpc.launch, mpc.rviz: Python MPC config for reference
- perception_dispatch.launch: method-selector for perception pipeline
- real_world_tmpc.launch: minimal real-robot launch (no Gazebo)

Key DOA fixes (submodule d7331f7):
- para_clipnode: feature-index alignment fix
- para_aggregate: passthrough modes for parallel SAM+CLIP
- model_manager: on-demand GPU model loading
- simulation.yaml: DISTANCE_THRESHOLD=1.0 rematch fix
- pointcloud_generator: real-world sensor tuning

Excluded (simulation only):
- exp/, FAPP/, onboard_detector/, pedestrian_simulator/
- pedsim_original/, jackal_simulator/
- Gazebo scene scripts and worlds
- mpc_planner/acados/ (349 MB pre-built lib, install separately)

Co-Authored-By: Claude Opus 4.7 <noreply@anthropic.com>

File: src/my_tb3_description/urdf_w_sensor/turtlebot3_burger.gazebo.xacro (robot description, xacro)
@@ -41,6 +41,6 @@
   </gazebo>
   <gazebo reference="wheel_left_link">
-    <mu1>0.1</mu1>
-    <mu2>0.1</mu2>
+    <mu1>1.0</mu1>
+    <mu2>1.0</mu2>
     <kp>500000.0</kp>
     <kd>10.0</kd>
@@ -51,6 +51,6 @@
   </gazebo>
   <gazebo reference="wheel_right_link">
-    <mu1>0.1</mu1>
-    <mu2>0.1</mu2>
+    <mu1>1.0</mu1>
+    <mu2>1.0</mu2>
     <kp>500000.0</kp>
     <kd>10.0</kd>
@@ -61,6 +61,6 @@
   </gazebo>
   <gazebo reference="caster_back_link">
-    <mu1>0.1</mu1>
-    <mu2>0.1</mu2>
+    <mu1>1.0</mu1>
+    <mu2>1.0</mu2>
     <kp>1000000.0</kp>
     <kd>100.0</kd>

File: src/my_tb3_description/urdf_w_sensor/turtlebot3_burger.urdf.xacro (robot description, xacro)
@@ -26,5 +26,5 @@
     </collision>
     <inertial>
-      <origin xyz="0 0 0" rpy="0 0 0"/>
+      <origin xyz="-0.02 0 -0.05" rpy="0 0 0"/>
       <mass value="8.2573504e-01"/>
       <inertia ixx="2.2124416e-03" ixy="-1.2294101e-05" ixz="3.4938785e-05"
